File: PCB/_autosave-PCRAMXpander.kicad_pcb (KiCad board)
At the start: 2 copper layers, 134.6 x 97.8 mm, 22 parts, among them J1 Bus_ISA_16bit, U1 ATF16V8B-15PU, U2 SN74LVCR16245ADGGR, U3 SN74LVC16244ADGGR, U4 SN74LVC16244ADGGR, U5 AS6C3216A-55TIN, U6 AS6C3216A-55TIN

Commit message: DRC clear
Routing:
- net +3.3V: track 356.6 -> 363.4 mm
- net BA01: track 57.1 -> 59.3 mm
- net BA14: track 31.9 -> 33.6 mm
- net BA15: track 34.3 -> 35.8 mm
- net BA16: track 35.0 -> 36.3 mm
- net BA02: track 54.4 -> 55.6 mm
- net A16: track 89.5 -> 90.2 mm
- net A17: track 114.2 -> 114.7 mm
- net GND: vias 166 -> 172
